Commit message: modify URDF mesh file directory for ros2

File: urdf/QUB.urdf (robot description, URDF)
Before this commit: robot QUB, 14 links, 13 joints
Links:
- link L_ankle_link: geometry visual mesh filename=package://QUB_gazebo/meshes/L_ankle_link.STL
- link L_calf_link: geometry visual mesh filename=package://QUB_gazebo/meshes/L_calf_link.STL
- link L_foot_link: geometry collision mesh filename=package://QUB_gazebo/meshes/collision/L_foot_link.STL; visual mesh filename=package://QUB_gazebo/meshes/L_foot_link.STL
- link L_hip_r_link: geometry visual mesh filename=package://QUB_gazebo/meshes/L_hip_r_link.STL
- link L_hip_y_link: geometry visual mesh filename=package://QUB_gazebo/meshes/L_hip_y_link.STL
- link L_thigh_link: geometry visual mesh filename=package://QUB_gazebo/meshes/L_thigh_link.STL
- link R_ankle_link: geometry visual mesh filename=package://QUB_gazebo/meshes/R_ankle_link.STL
- link R_calf_link: geometry visual mesh filename=package://QUB_gazebo/meshes/R_calf_link.STL
- link R_foot_link: geometry collision mesh filename=package://QUB_gazebo/meshes/collision/R_foot_link.STL; visual mesh filename=package://QUB_gazebo/meshes/R_foot_link.STL
- link R_hip_r_link: geometry visual mesh filename=package://QUB_gazebo/meshes/R_hip_r_link.STL
- link R_hip_y_link: geometry visual mesh filename=package://QUB_gazebo/meshes/R_hip_y_link.STL
- link R_thigh_link: geometry visual mesh filename=package://QUB_gazebo/meshes/R_thigh_link.STL
- link base_link: geometry collision box size=0.140 0.200 0.279; visual mesh filename=package://QUB_gazebo/meshes/base_link.STL
- link pelvis_link: geometry collision mesh filename=package://QUB_gazebo/meshes/collision/pelvis_link.STL; visual mesh filename=package://QUB_gazebo/meshes/pelvis_link.STL
